File: USB3/USB3pwr.kicad_sch (KiCad schematic)
At the start: 0 parts

Commit message: finished usb3.0
Parts:
- added C22, C46, C47, C48, C50, C51, C52, C53, C54, C55, C56: 0.1uF, symbol Device:C
- added C49, C57, C59: 10uF, symbol Device:C
- added C58: 220uF, symbol Device:C
- added FB5, FB6: 220 @ 100MHZ, symbol Device:FerriteBead
- added R21: 10k, symbol Device:R
- added U7: TPS74611PQWDRBRQ1, Package_SON:VSON-8-1EP_3x3mm_P0.65mm_EP1.65x2.4mm_ThermalVias, symbol Regulator_Linear:LM1117LD-1.8
Connections:
- new net: C58.1, FB6.2, R21.1, U7.1 (OUT)
- new net: R21.2, U7.6 (PG)
- new net +1.8v_(Output): C59.1, U7.5 (EN), U7.8 (IN)
- new net GND: C22.1, C46.1, C47.1, C48.1, C49.1, C50.2, C51.2, C52.2, C53.2, C54.2, C55.2, C56.2, C57.2, C58.2, C59.2, U7.4 (GND)
- new net USB_3V3: FB5.2
- new net VDD: C50.1, C51.1, C52.1, C53.1, C54.1, C55.1, C56.1, C57.1, FB6.1
- new net VDD33: C22.2, C46.2, C47.2, C48.2, C49.2, FB5.1
