File: USB3/USB3down12.kicad_sch (KiCad schematic)
At the start: 0 parts

Commit message: usb3 down done
Parts:
- added C10, C11, C15, C16: 0.1uF 0201, symbol Device:C
- added C12, C14, C17, C24: 0.1uF, symbol Device:C
- added C13, C18: 0.001uF, symbol Device:C
- added D10, D11, D12, D13, D14, D3, D4, D5, D6, D7, D8, D9: ESD5311N-2/TR, Diode_SMD:Infineon_SG-WLL-2-3_0.58x0.28_P0.36mm, symbol Diode:ESD131-B1-W0201
- added FB1, FB2: 220 @ 100Mhz, symbol Device:FerriteBead
- added FL2, FL3: MCZ1210AH900L2TD0G, symbol Filter:Choke_CommonMode_FerriteCore_1423
- added P1, P2: USB_C_Plug, symbol Connector:USB_C_Plug
- added R8, R9: 1M 0402, symbol Device:R
Connections:
- new net: C17.1, FB2.2, P2.A4 (VBUS), P2.A9 (VBUS), P2.B4 (VBUS), P2.B9 (VBUS)
- new net: D6.1 (A1), FL2.3, P1.A6 (D+)
- new net: D5.1 (A1), FL2.4, P1.A7 (D-)
- new net: C15.1, D13.1 (A1), P2.A3 (TX1-), P2.B3 (TX2-)
- new net: C16.2, D14.1 (A1), P2.A2 (TX1+), P2.B2 (TX2+)
- new net: D12.1 (A1), FL3.3, P2.A6 (D+)
- new net: D11.1 (A1), FL3.4, P2.A7 (D-)
- new net: C11.2, D8.1 (A1), P1.A2 (TX1+), P1.B2 (TX2+)
- new net: C12.1, FB1.2, P1.A4 (VBUS), P1.A9 (VBUS), P1.B4 (VBUS), P1.B9 (VBUS)
- new net: C10.1, D7.1 (A1), P1.A3 (TX1-), P1.B3 (TX2-)
- new net DN1_VBUS: FB1.1
- new net DN2_VBUS: FB2.1
- new net GND: C12.2, C13.2, C14.2, C17.2, C18.2, C24.2, D10.2 (A2), D11.2 (A2), D12.2 (A2), D13.2 (A2), D14.2 (A2), D3.2 (A2), D4.2 (A2), D5.2 (A2), D6.2 (A2), D7.2 (A2), D8.2 (A2), D9.2 (A2), P1.A1 (GND), P1.A12 (GND), P1.B1 (GND), P1.B12 (GND), P2.A1 (GND), P2.A12 (GND), P2.B1 (GND), P2.B12 (GND), R8.2, R9.2
- new net GNDPWR: C13.1, C14.1, C18.1, C24.1, P1.S1 (SHIELD), P2.S1 (SHIELD), R8.1, R9.1
- new net USB_DM_DN1: FL2.1
- new net USB_DM_DN2: FL3.1
- new net USB_DP_DN1: FL2.2
- new net USB_DP_DN2: FL3.2
- new net USB_SSRXM_DN1: D3.1 (A1), P1.A10 (RX2-), P1.B10 (RX1-)
- new net USB_SSRXM_DN2: D9.1 (A1), P2.A10 (RX2-), P2.B10 (RX1-)
- new net USB_SSRXP_DN1: D4.1 (A1), P1.A11 (RX2+), P1.B11 (RX1+)
- new net USB_SSRXP_DN2: D10.1 (A1), P2.A11 (RX2+), P2.B11 (RX1+)
- new net USB_SSTXM_DN1: C10.2
- new net USB_SSTXM_DN2: C15.2
- new net USB_SSTXP_DN1: C11.1
- new net USB_SSTXP_DN2: C16.1

Commit message: Ethernet and MIPI cam done, USBC OTG started
Parts:
- D10, D11, D12, D13, D14, D3, D4, D5, D6, D7, D8, D9: footprint Diode_SMD:Infineon_SG-WLL-2-3_0.58x0.28_P0.36mm -> radxa:DFN1006-2L
Changed lines of the file:
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@@
 			)
 		)
-		(property "Footprint" "Diode_SMD:Infineon_SG-WLL-2-3_0.58x0.28_P0.36mm"
+		(property "Footprint" "radxa:DFN1006-2L"
 			(at 69.85 181.61 0)
 			(effects
@@
 			)
 		)
-		(property "Footprint" "Diode_SMD:Infineon_SG-WLL-2-3_0.58x0.28_P0.36mm"
+		(property "Footprint" "radxa:DFN1006-2L"
 			(at 109.22 92.71 0)
 			(effects
@@
 			)
 		)
-		(property "Footprint" "Diode_SMD:Infineon_SG-WLL-2-3_0.58x0.28_P0.36mm"
+		(property "Footprint" "radxa:DFN1006-2L"
 			(at 132.08 92.71 0)
 			(effects
@@
 			)
 		)
-		(property "Footprint" "Diode_SMD:Infineon_SG-WLL-2-3_0.58x0.28_P0.36mm"
+		(property "Footprint" "radxa:DFN1006-2L"
 			(at 81.28 181.61 0)
 			(effects
@@
 			)
 		)
-		(property "Footprint" "Diode_SMD:Infineon_SG-WLL-2-3_0.58x0.28_P0.36mm"
+		(property "Footprint" "radxa:DFN1006-2L"
 			(at 86.36 92.71 0)
 			(effects
@@
 			)
 		)
-		(property "Footprint" "Diode_SMD:Infineon_SG-WLL-2-3_0.58x0.28_P0.36mm"
+		(property "Footprint" "radxa:DFN1006-2L"
 			(at 35.56 181.61 0)
 			(effects
@@
 			)
 		)
-		(property "Footprint" "Diode_SMD:Infineon_SG-WLL-2-3_0.58x0.28_P0.36mm"
+		(property "Footprint" "radxa:DFN1006-2L"
 			(at 120.65 92.71 0)
 			(effects
@@
 			)
 		)
-		(property "Footprint" "Diode_SMD:Infineon_SG-WLL-2-3_0.58x0.28_P0.36mm"
+		(property "Footprint" "radxa:DFN1006-2L"
 			(at 46.99 181.61 0)
 			(effects
@@
 			)
 		)
-		(property "Footprint" "Diode_SMD:Infineon_SG-WLL-2-3_0.58x0.28_P0.36mm"
+		(property "Footprint" "radxa:DFN1006-2L"
 			(at 24.13 181.61 0)
 			(effects
@@
 			)
 		)
-		(property "Footprint" "Diode_SMD:Infineon_SG-WLL-2-3_0.58x0.28_P0.36mm"
+		(property "Footprint" "radxa:DFN1006-2L"
 			(at 74.93 92.71 0)
 			(effects
@@
 			)
 		)
-		(property "Footprint" "Diode_SMD:Infineon_SG-WLL-2-3_0.58x0.28_P0.36mm"
+		(property "Footprint" "radxa:DFN1006-2L"
 			(at 58.42 181.61 0)
 			(effects
@@
 			)
 		)
-		(property "Footprint" "Diode_SMD:Infineon_SG-WLL-2-3_0.58x0.28_P0.36mm"
+		(property "Footprint" "radxa:DFN1006-2L"
 			(at 97.79 92.71 0)
 			(effects

Commit message: usbc work
Parts:
- FL2, FL3: value MCZ1210AH900L2TD0G -> MCZ1210DH120L2TA0G
Changed lines of the file:
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@@
 			)
 		)
-		(property "Value" "MCZ1210AH900L2TD0G"
+		(property "Value" "MCZ1210DH120L2TA0G"
 			(at 96.393 33.02 0)
 			(effects
@@
 			)
 		)
-		(property "Value" "MCZ1210AH900L2TD0G"
+		(property "Value" "MCZ1210DH120L2TA0G"
 			(at 45.593 121.92 0)
 			(effects
