File: USB3/USB3down34.kicad_sch (KiCad schematic)
At the start: 0 parts

Commit message: usb3 down done
Parts:
- added C25, C26, C28, C29: 0.1uF 0201, symbol Device:C
- added C27, C31, C32, C34: 0.1uF, symbol Device:C
- added C30, C33: 0.001uF, symbol Device:C
- added D15, D16, D17, D18, D19, D20, D21, D22, D23, D24, D25, D26: ESD5311N-2/TR, Diode_SMD:Infineon_SG-WLL-2-3_0.58x0.28_P0.36mm, symbol Diode:ESD131-B1-W0201
- added FB3, FB4: 220 @ 100Mhz, symbol Device:FerriteBead
- added FL4, FL5: MCZ1210AH900L2TD0G, symbol Filter:Choke_CommonMode_FerriteCore_1423
- added P3, P4: USB_C_Plug, symbol Connector:USB_C_Plug
- added R10, R11: 1M 0402, symbol Device:R
Connections:
- new net: C29.2, D26.1 (A1), P4.A2 (TX1+), P4.B2 (TX2+)
- new net: D18.1 (A1), FL4.3, P3.A6 (D+)
- new net: D17.1 (A1), FL4.4, P3.A7 (D-)
- new net: C28.1, D25.1 (A1), P4.A3 (TX1-), P4.B3 (TX2-)
- new net: C31.1, FB4.2, P4.A4 (VBUS), P4.A9 (VBUS), P4.B4 (VBUS), P4.B9 (VBUS)
- new net: C27.1, FB3.2, P3.A4 (VBUS), P3.A9 (VBUS), P3.B4 (VBUS), P3.B9 (VBUS)
- new net: D24.1 (A1), FL5.3, P4.A6 (D+)
- new net: C25.1, D19.1 (A1), P3.A3 (TX1-), P3.B3 (TX2-)
- new net: C26.2, D21.1 (A1), P3.A2 (TX1+), P3.B2 (TX2+)
- new net: D23.1 (A1), FL5.4, P4.A7 (D-)
- new net DN3_VBUS: FB4.1
- new net DN4_VBUS: FB3.1
- new net GND: C27.2, C30.2, C31.2, C32.2, C33.2, C34.2, D15.2 (A2), D16.2 (A2), D17.2 (A2), D18.2 (A2), D19.2 (A2), D20.2 (A2), D21.2 (A2), D22.2 (A2), D23.2 (A2), D24.2 (A2), D25.2 (A2), D26.2 (A2), P3.A1 (GND), P3.A12 (GND), P3.B1 (GND), P3.B12 (GND), P4.A1 (GND), P4.A12 (GND), P4.B1 (GND), P4.B12 (GND), R10.2, R11.2
- new net GNDPWR: C30.1, C32.1, C33.1, C34.1, P3.S1 (SHIELD), P4.S1 (SHIELD), R10.1, R11.1
- new net USB_DM_DN3: FL5.1
- new net USB_DM_DN4: FL4.1
- new net USB_DP_DN3: FL5.2
- new net USB_DP_DN4: FL4.2
- new net USB_SSRXM_DN3: D20.1 (A1), P4.A10 (RX2-), P4.B10 (RX1-)
- new net USB_SSRXM_DN4: D15.1 (A1), P3.A10 (RX2-), P3.B10 (RX1-)
- new net USB_SSRXP_DN3: D22.1 (A1), P4.A11 (RX2+), P4.B11 (RX1+)
- new net USB_SSRXP_DN4: D16.1 (A1), P3.A11 (RX2+), P3.B11 (RX1+)
- new net USB_SSTXM_DN3: C28.2
- new net USB_SSTXM_DN4: C25.2
- new net USB_SSTXP_DN3: C29.1
- new net USB_SSTXP_DN4: C26.1

Commit message: Ethernet and MIPI cam done, USBC OTG started
Parts:
- D15, D16, D17, D18, D19, D20, D21, D22, D23, D24, D25, D26: footprint Diode_SMD:Infineon_SG-WLL-2-3_0.58x0.28_P0.36mm -> radxa:DFN1006-2L
Changed lines of the file:
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@@
 			)
 		)
-		(property "Footprint" "Diode_SMD:Infineon_SG-WLL-2-3_0.58x0.28_P0.36mm"
+		(property "Footprint" "radxa:DFN1006-2L"
 			(at 58.42 182.88 0)
 			(effects
@@
 			)
 		)
-		(property "Footprint" "Diode_SMD:Infineon_SG-WLL-2-3_0.58x0.28_P0.36mm"
+		(property "Footprint" "radxa:DFN1006-2L"
 			(at 35.56 182.88 0)
 			(effects
@@
 			)
 		)
-		(property "Footprint" "Diode_SMD:Infineon_SG-WLL-2-3_0.58x0.28_P0.36mm"
+		(property "Footprint" "radxa:DFN1006-2L"
 			(at 46.99 182.88 0)
 			(effects
@@
 			)
 		)
-		(property "Footprint" "Diode_SMD:Infineon_SG-WLL-2-3_0.58x0.28_P0.36mm"
+		(property "Footprint" "radxa:DFN1006-2L"
 			(at 74.93 93.98 0)
 			(effects
@@
 			)
 		)
-		(property "Footprint" "Diode_SMD:Infineon_SG-WLL-2-3_0.58x0.28_P0.36mm"
+		(property "Footprint" "radxa:DFN1006-2L"
 			(at 24.13 182.88 0)
 			(effects
@@
 			)
 		)
-		(property "Footprint" "Diode_SMD:Infineon_SG-WLL-2-3_0.58x0.28_P0.36mm"
+		(property "Footprint" "radxa:DFN1006-2L"
 			(at 86.36 93.98 0)
 			(effects
@@
 			)
 		)
-		(property "Footprint" "Diode_SMD:Infineon_SG-WLL-2-3_0.58x0.28_P0.36mm"
+		(property "Footprint" "radxa:DFN1006-2L"
 			(at 120.65 93.98 0)
 			(effects
@@
 			)
 		)
-		(property "Footprint" "Diode_SMD:Infineon_SG-WLL-2-3_0.58x0.28_P0.36mm"
+		(property "Footprint" "radxa:DFN1006-2L"
 			(at 109.22 93.98 0)
 			(effects
@@
 			)
 		)
-		(property "Footprint" "Diode_SMD:Infineon_SG-WLL-2-3_0.58x0.28_P0.36mm"
+		(property "Footprint" "radxa:DFN1006-2L"
 			(at 69.85 182.88 0)
 			(effects
@@
 			)
 		)
-		(property "Footprint" "Diode_SMD:Infineon_SG-WLL-2-3_0.58x0.28_P0.36mm"
+		(property "Footprint" "radxa:DFN1006-2L"
 			(at 97.79 93.98 0)
 			(effects
@@
 			)
 		)
-		(property "Footprint" "Diode_SMD:Infineon_SG-WLL-2-3_0.58x0.28_P0.36mm"
+		(property "Footprint" "radxa:DFN1006-2L"
 			(at 81.28 182.88 0)
 			(effects
@@
 			)
 		)
-		(property "Footprint" "Diode_SMD:Infineon_SG-WLL-2-3_0.58x0.28_P0.36mm"
+		(property "Footprint" "radxa:DFN1006-2L"
 			(at 132.08 93.98 0)
 			(effects

Commit message: usbc work
Parts:
- FL4, FL5: value MCZ1210AH900L2TD0G -> MCZ1210DH120L2TA0G
Changed lines of the file:
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@@
 			)
 		)
-		(property "Value" "MCZ1210AH900L2TD0G"
+		(property "Value" "MCZ1210DH120L2TA0G"
 			(at 45.593 123.19 0)
 			(effects
@@
 			)
 		)
-		(property "Value" "MCZ1210AH900L2TD0G"
+		(property "Value" "MCZ1210DH120L2TA0G"
 			(at 96.393 34.29 0)
 			(effects
