File: RJ45.kicad_sch (KiCad schematic)
At the start: 0 parts

Commit message: Ethernet and MIPI cam done, USBC OTG started
Parts:
- added C60: 0.1uF 16v, symbol Device:C
- added D27, D28: ESD5311N-2/TR, radxa:DFN1006-2L, symbol Diode:ESD131-B1-W0201
- added J2: LPJG0926HENL, radxa:LPJG0926HENL, symbol LPJG0926HENL:LPJG0926HENL
- added J3: Conn_02x02_Odd_Even, symbol Connector_Generic:Conn_02x02_Odd_Even
- added R29, R30: 510R, symbol Device:R
- added U8, U9: ~, radxa:ESD5344-D, symbol raxda:ESD5344-D
Connections:
- new net: C60.2, J2.5 (TD2-_2), J2.6 (TD2-_3)
- new net: J2.17 (A_YELLOW), R30.2
- new net: J2.11 (VC1), J3.2 (Pin_2)
- new net: J2.12 (VC2), J3.1 (Pin_1)
- new net: J2.13 (VC3), J3.4 (Pin_4)
- new net: J2.14 (VC4), J3.3 (Pin_3)
- new net: J2.15 (A_GREEN), R29.1
- new net Ethernet_Pair0_N: J2.2 (TD1-), U8. (IO2), U8.9 (NC9)
- new net Ethernet_Pair0_P: J2.1 (TD1+), U8.1 (IO1), U8.10 (NC10)
- new net Ethernet_Pair1_N: J2.4 (TD2-_1), U8.5 (IO4), U8.6 (NC6)
- new net Ethernet_Pair1_P: J2.3 (TD2+), U8.4 (IO3), U8.7 (NC7)
- new net Ethernet_Pair2_N: J2.8 (TD3-), U9. (IO2), U9.9 (NC9)
- new net Ethernet_Pair2_P: J2.7 (TD3+), U9.1 (IO1), U9.10 (NC10)
- new net Ethernet_Pair3_N: J2.10 (TD4-), U9.5 (IO4), U9.6 (NC6)
- new net Ethernet_Pair3_P: J2.9 (TD4+), U9.4 (IO3), U9.7 (NC7)
- new net Ethernet_nLED2(3.3v): D28.2 (A2), R29.2
- new net Ethernet_nLED3(3.3v): D27.1 (A1), R30.1
- new net GND: C60.1, D27.2 (A2), D28.1 (A1), J2.16 (K_GREEN), J2.18 (K_YELLOW), J2.19 (MH3), J2.20 (MH4), U8.3 (GND), U8.8 (GND), U9.3 (GND), U9.8 (GND)
