File: USBC.kicad_sch (KiCad schematic)
At the start: 2 parts, among them J5 USB_C_Receptacle, U11 FUSB302BMPX

Commit message: usbc work
Parts:
- added C63, C64, C65, C66, C67, C68: 0.1uF, symbol Device:C
- added FL6: MCZ1210DH120L2TA0G, symbol Filter:Choke_CommonMode_FerriteCore_1423
- added R31, R32: 2.2R, symbol Device:R
- added R33, R34: 100K, symbol Device:R
- added R35, R36: 2M, symbol Device:R
- added U12, U13: TPD4E05U06DQA, Package_SON:USON-10_2.5x1.0mm_P0.5mm, symbol Power_Protection:TPD4E05U06DQA
Connections:
- net TYPEC0_SBU1: now also C67.2
- net TYPEC0_SBU2: now also C68.2
- net TYPEC0_SSRX1N: now also J5.B10 (RX1-), U12.5 (D2-)
- net TYPEC0_SSRX1P: now also J5.B11 (RX1+), U12.4 (D2+)
- net TYPEC0_SSRX2N: now also J5.A10 (RX2-), U13.5 (D2-)
- net TYPEC0_SSRX2P: now also J5.A11 (RX2+), U13.4 (D2+)
- net TYPEC0_SSTX1N: now also C63.1
- net TYPEC0_SSTX1P: now also C65.1
- net TYPEC0_SSTX2N: now also C64.1
- net TYPEC0_SSTX2P: now also C66.1
- net GND: now reaches J5.A1 (GND), J5.A12 (GND), J5.B1 (GND), J5.B12 (GND)
- net GND: now also J5.S1 (SHIELD), R35.1, R36.1, U12.3 (GND), U12.8 (GND), U13.3 (GND), U13.8 (GND)
- net at J5.A2 (TX1+): now also C65.2, U12.1 (D1+)
- net at J5.A3 (TX1-): now also C63.2, U12.2 (D1-)
- net at J5.A6 (D+): now also J5.B6 (D+), FL6.2
- net at J5.A7 (D-): now also J5.B7 (D-), FL6.1
- net at J5.A8 (SBU1): now also C67.1, R33.2, R35.2
- net at J5.B2 (TX2+): now also C66.2, U13.1 (D1+)
- net at J5.B3 (TX2-): now also C64.2, U13.2 (D1-)
- net at J5.B8 (SBU2): now also C68.1, R34.2, R36.2
- new net: FL6.3, R32.1
- new net: FL6.4, R31.1
- new net GPIO_3V3_3: R33.1
- new net GPIO_3V3_4: R34.1
- new net USB2_N: R31.2
- new net USB2_P: R32.2
Other:
- moved on the sheet: U11

Commit message: usbc work
Parts:
- added C69, C72: 22uF, symbol Device:C_Polarized
- added C70, C71: 0.1uF, symbol Device:C_Polarized
- added R38: 100K, symbol Device:R
- added R39: 4.7K, symbol Device:R
- added U14: Silergy SY6280AAC, symbol raxda:SGM2576YN5G/TR
Connections:
- net GND: now also C69.2, C70.2, C71.2, C72.2, R38.2, R39.2, U14.2 (GND)
- net at J5.A5 (CC1): now also U11.10 (CC1), U11.11 (CC1)
- net at J5.B5 (CC2): now also U11.1 (CC2), U11.14 (CC2)
- new net: R39.1, U14.3 (OCB)
- new net: C70.1, C72.1, U14.1 (VOUT)
- new net TYPEC5V_PWREN_H: R38.1, U14.4 (EN)
- new net VCC5V0_SYS: C69.1, C71.1, U14.5 (IN)
Other:
- moved on the sheet: U11

Commit message: usbc done, replaced pcb with radxa example
Parts:
- added C73: 1uF, symbol Device:C
- added C74, C75: 0.1uF, symbol Device:C
- added C76, C77: 220pF, symbol Device:C
- added C78: 22uF 25V, symbol Device:C
- added C79: 10uF 25V, symbol Device:C
- added D29: BZT52C15, symbol BZT52C15:Diode
- added D30, D31, D32, D33, D34, D35: ESD5311N-2/TR, radxa:DFN1006-2L, symbol Diode:ESD131-B1-W0201
- added R37: 4.7K, symbol Device:R
- C69, C70, C71, C72: symbol Device:C_Polarized -> Device:C
Connections:
- net GND: now also U11.15 (GND), U11.8 (GND), U11.9 (GND), C73.1, C74.1, C75.1, C76.2, C77.2, C78.2, C79.2, D29.1 (A), D30.1 (A1), D31.1 (A1), D32.2 (A2), D33.2 (A2), D34.2 (A2), D35.2 (A2)
- net VCC5V0_SYS: now also C70.1, C72.1, U11.12 (VCONN), U11.13 (VCONN), C73.2, C74.2; no longer C69.1, C71.1
- net at C67.1, J5.A8 (SBU1), R33.2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: now also D30.2 (A2)
- net at J5.A4 (VBUS), J5.A9 (VBUS), J5.B4 (VBUS)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: now also C69.1, C71.1, U11.2 (VBUS), U14.1 (VOUT), C78.1, C79.1, D29.2 (C)
- net at J5.A5 (CC1), U11.10 (CC1), U11.11 (CC1): now also C77.1, D32.1 (A1)
- net at FL6.2, J5.A6 (D+), J5.B6 (D+): now also D35.1 (A1)
- net at FL6.1, J5.A7 (D-), J5.B7 (D-): now also D34.1 (A1)
- net at J5.B5 (CC2), U11.1 (CC2), U11.14 (CC2): now also C76.1, D33.1 (A1)
- net at C68.1, J5.B8 (SBU2), R34.2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: now also D31.2 (A2)
- net +3.3v_(Output): now reaches U11.3 (VDD), U11.4 (VDD)
- net +3.3v_(Output): now also C75.2, R37.1
- net GPIO_3V3_CC_INT0_L: now reaches U11.5 (INT_N)
- net GPIO_3V3_CC_INT0_L: now also R37.2
- net I2C_SCL_3V3: now reaches U11.6 (SCL)
- net I2C_SDA_3V3: now reaches U11.7 (SDA)
Other:
- moved on the sheet: R38, R39, U14
